Commit message: fix: restore H2 right hand visual

File: models/unitree/h2/urdf/robot.urdf (robot description, URDF)
Before this commit: robot H2, 34 links, 33 joints
Links:
- link right_hand_link: geometry collision mesh filename=meshes/right_hand_link.stl; visual mesh filename=meshes/right_hand_link.stl
